File: hardware/kicad/alimentazione.kicad_sch (KiCad schematic)
At the start: 18 parts, among them J8 12V DC, U10 L78L05, U11 AP63205WU

Commit message: rev 0.3: front panel with I2C OLED, encoder and OUTPUT button
PCF8574 expander (0x20) with INT on GPIO0, 10-pin IDC connector,
RC debounce, I2C pull-ups 2.2k, re-routed PCB (DRC/parity clean),
updated BOM, slides (front panel page) and README.

Co-Authored-By: Claude Opus 5.5 <noreply@anthropic.com>
Claude-Session: https://claude.ai/code/session_013KrwoEq2Y4F9LNKutY5RJ4
Parts:
- removed C28, C31, C32: 10u 25V, Capacitor_SMD:C_1206_3216Metric, symbol Device:C
- removed C29: 100n, Capacitor_SMD:C_1206_3216Metric, symbol Device:C
- removed C30: 1u, Capacitor_SMD:C_1206_3216Metric, symbol Device:C
- removed C33, C34: 100n 50V, Capacitor_SMD:C_1206_3216Metric, symbol Device:C
- removed J8: 12V DC, Connector_BarrelJack:BarrelJack_Horizontal, symbol Connector:Barrel_Jack
- removed R49: 1k5, Resistor_SMD:R_1206_3216Metric, symbol Device:R
- removed R50: 100k, Resistor_SMD:R_1206_3216Metric, symbol Device:R
- removed U10: L78L05, Package_SO:SOIC-8_3.9x4.9mm_P1.27mm, symbol Regulator_Linear:L78L05_SO8
- removed U11: AP63205WU, Package_TO_SOT_SMD:TSOT-23-6, symbol Regulator_Switching:AP63205WU
- added C37: 1u, Capacitor_SMD:C_1206_3216Metric, symbol Device:C
- added C38, C39: 10u 25V, Capacitor_SMD:C_1206_3216Metric, symbol Device:C
- added C40, C41: 100n 50V, Capacitor_SMD:C_1206_3216Metric, symbol Device:C
- added C42, C43: 22u 10V, Capacitor_SMD:C_1206_3216Metric, symbol Device:C
- added J9: 12V DC, Connector_BarrelJack:BarrelJack_Horizontal, symbol Connector:Barrel_Jack
- added R54: 1k5, Resistor_SMD:R_1206_3216Metric, symbol Device:R
- added R55: 100k, Resistor_SMD:R_1206_3216Metric, symbol Device:R
- added U11: L78L05, Package_SO:SOIC-8_3.9x4.9mm_P1.27mm, symbol Regulator_Linear:L78L05_SO8
- added U12: AP63205WU, Package_TO_SOT_SMD:TSOT-23-6, symbol Regulator_Switching:AP63205WU
- C35: value 22u 10V -> 10u 25V
- C36: value 22u 10V -> 100n
Connections:
- net +12V: now also C35.1, C36.1, C39.1, C40.1, R55.1, U11.8 (IN), U12.3 (IN)
- net +3V3: now also C38.1, R54.1
- net +5V: now also C37.1, U11.1 (OUT)
- net +5V_WIFI: now also C42.1, C43.1, U12.1 (FB); no longer C35.1, C36.1
- net BUCK_BST: now also C41.1, U12.6 (BST)
- net BUCK_EN: now also R55.2, U12.2 (EN)
- net BUCK_SW: now also C41.2, U12.5 (SW)
- net GND: now also C37.2, C38.2, C39.2, C40.2, C42.2, C43.2, J9.2, U11.2 (GND), U11.3 (GND), U11.6 (GND), U11.7 (GND), U12.4 (GND)
- net at D4.2 (A): now also J9.1
- net at D5.2 (A): now also R54.2
