File: hardware/kicad/controllo.kicad_sch (KiCad schematic)
At the start: 29 parts, among them J4 D1mini SX, J5 D1mini DX, J6 FAN, J7 NTC, Q5 FDS9926A, Q6 FDS9926A, Q7 FDS9926A, U9 DAC8565

Commit message: rev 0.3: front panel with I2C OLED, encoder and OUTPUT button
PCF8574 expander (0x20) with INT on GPIO0, 10-pin IDC connector,
RC debounce, I2C pull-ups 2.2k, re-routed PCB (DRC/parity clean),
updated BOM, slides (front panel page) and README.

Co-Authored-By: Claude Opus 5.5 <noreply@anthropic.com>
Claude-Session: https://claude.ai/code/session_013KrwoEq2Y4F9LNKutY5RJ4
Parts:
- removed J6: FAN, Connector_Molex:Molex_KK-254_AE-6410-04A_1x04_P2.54mm_Vertical, symbol Connector_Generic:Conn_01x04
- removed U9: DAC8565, Package_SO:TSSOP-16_4.4x5mm_P0.65mm, symbol Analog_DAC:DAC8565
- added C28, C29, C30, C32, C33, C34: 100n, Capacitor_SMD:C_1206_3216Metric, symbol Device:C
- added C31: 1u, Capacitor_SMD:C_1206_3216Metric, symbol Device:C
- added J6: FRONT PANEL, Connector_IDC:IDC-Header_2x05_P2.54mm_Vertical, symbol Connector_Generic:Conn_02x05_Odd_Even
- added J8: NTC, Connector_Molex:Molex_KK-254_AE-6410-04A_1x04_P2.54mm_Vertical, symbol Connector_Generic:Conn_01x04
- added R49: 100R, Resistor_SMD:R_1206_3216Metric, symbol Device:R
- added R50: 100k, Resistor_SMD:R_1206_3216Metric, symbol Device:R
- added R51: 10k, Resistor_SMD:R_1206_3216Metric, symbol Device:R
- added R52, R53: 10k 0.1%, Resistor_SMD:R_1206_3216Metric, symbol Device:R
- added U10: DAC8565, Package_SO:TSSOP-16_4.4x5mm_P0.65mm, symbol Analog_DAC:DAC8565
- added U9: PCF8574T, Package_SO:SOIC-16W_7.5x10.3mm_P1.27mm, symbol Interface_Expansion:PCF8574T
- C23, C25, C26: value 100n -> 10n; Note (none) -> Antirimbalzo 100 us
- C24: value 1u -> 10n; Note (none) -> Antirimbalzo 100 us
- C27: value 100n -> 10u 25V; Note (none) -> Disaccoppiamento OLED
- J5: Note TX RX(GPIO3) D1(5) D2(4) D3(0) D4(2) G 5V; GPIO0/2/15 = str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 -> TX RX(GPIO3) D1(5) D2(4) D3(0)=INT espansore D4(2) G 5V; GP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
- J7: value NTC -> FAN; Note 2x NTC 10k B3950 incollate allo spreader -> Ventola 12 V 4 fili (cooler SP3/TR4)
- R37: value 4k7 -> 2k2; Note (none) -> Bus esteso al pannello frontale (rev 0.3)
- R38: value 4k7 -> 2k2
- R40: value 1k -> 10k
- R41: Note Pull-down: ARM basso = carico disabilitato -> (none)
- R42: value 100k -> 10k; Note Lettura ARM: 100k, un GPIO pilotato al boot non puo armare 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 -> (none)
- R43: value 10k -> 470R; Note (none) -> LED OUTPUT sul pannello: anodo a 3V3, catodo qui
- R44: value 100R -> 10k
- R45: value 100k -> 1k
- R46: Note (none) -> Pull-down: ARM basso = carico disabilitato
- R47: value 10k 0.1% -> 100k; Note (none) -> Lettura ARM: 100k, un GPIO pilotato al boot non puo armare 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
- R48: value 10k 0.1% -> 10k; Note NTC2 di riserva: il D1 mini ha un solo ADC (A0 = NTC1) -> (none)
Connections:
- net +12V: now also J7.2 (Pin_2)
- net +3V3: now also C22.1, C27.1, R40.1, R41.1, R42.1, R44.1, C28.1, C32.1, J6.1 (Pin_1), R51.1, R52.1, R53.1, U10.12 (IOVDD), U9.16 (VDD); no longer C25.1, R46.1, R47.1, R48.1
- net +5V: now also R48.1, C30.1, C31.1, U10.4 (AVDD); no longer C23.1, C24.1, R43.1
- net ARM: now also R45.2, R46.1, R47.1; no longer R40.2, R41.1, R42.1
- net ARM_DRV: now also R45.1; no longer R40.1
- net ARM_FB: now also R47.2; no longer R42.2
- net CLAMP: now also R48.2; no longer R43.2
- net DAC_A: now also U10.1 (VOUTA)
- net DAC_B: now also U10.2 (VOUTB)
- net DAC_C: now also U10.7 (VOUTC)
- net DAC_D: now also U10.8 (VOUTD)
- net DAC_RST: now also R44.2, U10.13 (~{RST}); no longer R39.2
- net DAC_SYNC: now also U10.9 (~{SYNC})
- net DAC_VREF: now also C29.1, U10.3 (VREFH/VREFOUT); no longer C22.1
- net FAN_PWM: now also J7.4 (Pin_4)
- net FAN_PWM_G: now also R49.2, R50.1; no longer R44.2, R45.1
- net FAN_PWM_MCU: now also R49.1; no longer R44.1
- net FAN_TACH: now also J7.3 (Pin_3), R51.2; no longer R46.2
- net GND: now also J7.1 (Pin_1), R46.2, C28.2, C29.2, C30.2, C31.2, C32.2, C33.2, C34.2, J6.2 (Pin_2), J6.4 (Pin_4), J8.2 (Pin_2), J8.4 (Pin_4), R50.2, U10.14 (RSTSEL), U10.15 (~{ENABLE}), U10.16 (LDAC), U10.5 (VREFL), U10.6 (GND), U9.1 (A0), U9.2 (A1), U9.3 (A2), U9.8 (GND); no longer J7.2 (Pin_2), J7.4 (Pin_4), R41.2, R45.2
- net I2C_SCL: now also J6.5 (Pin_5), U9.14 (SCL)
- net I2C_SDA: now also J6.3 (Pin_3), U9.15 (SDA)
- net NTC1: now also C33.1, J8.1 (Pin_1), R52.2; no longer C26.1, J7.1 (Pin_1), R47.2
- net NTC2: now also C34.1, J8.3 (Pin_3), R53.2; no longer C27.1, J7.3 (Pin_3), R48.2
- net SPI_MOSI: now also U10.11 (DIN)
- net SPI_SCK: now also U10.10 (SCLK)
- net EXP_INT: now reaches J5.5 (Pin_5)
- net EXP_INT: now also U9.13 (~{INT})
- new net FP_BTN_OUT: C26.1, J6.9 (Pin_9), R42.2, U9.7 (P3)
- new net FP_ENC_A: C23.1, J6.6 (Pin_6), R39.2, U9.4 (P0)
- new net FP_ENC_B: C24.1, J6.7 (Pin_7), R40.2, U9.5 (P1)
- new net FP_ENC_SW: C25.1, J6.8 (Pin_8), R41.2, U9.6 (P2)
- new net FP_LED: J6.10 (Pin_10), R43.2
- new net PCF_LED: R43.1, U9.9 (P4)
- no-connect marks 3 -> 5
Other:
- note added: "Pannello frontale: OLED I2C, encoder con pulsante, tasto OUTPUT (rev 0.3)"
