File: hardware/kicad/control.kicad_sch (KiCad schematic)
At the start: 43 parts, among them J4 D1mini SX, J5 D1mini DX, J6 FRONT PANEL, J7 FAN, J8 NTC, Q5 FDS9926A, Q6 FDS9926A, Q7 FDS9926A, U10 DAC8565, U9 PCF8574T

Commit message: Translate schematic and PCB to English
Sheets renamed (input, channels, control, power), all titles, notes,
values and board texts in English; symbol library renamed to eload.
Re-routed board: DRC with schematic parity clean.

Co-Authored-By: Claude Opus 5.5 <noreply@anthropic.com>
Claude-Session: https://claude.ai/code/session_013KrwoEq2Y4F9LNKutY5RJ4
Parts:
- C23, C24, C25, C26: Note Antirimbalzo 100 us -> Debounce 100 us
- C27: Note Disaccoppiamento OLED -> OLED decoupling
- J4: value D1mini SX -> D1mini L; Note RST A0 D0(GPIO16) D5(14) D6(12) D7(13) D8(15) 3V3; il 3V3 d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 -> RST A0 D0(GPIO16) D5(14) D6(12) D7(13) D8(15) 3V3; the modu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
- J5: value D1mini DX -> D1mini R; Note TX RX(GPIO3) D1(5) D2(4) D3(0)=INT espansore D4(2) G 5V; GP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 -> TX RX(GPIO3) D1(5) D2(4) D3(0)=expander INT D4(2) G 5V; GPI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
- J6: Note Flat 10 poli verso il pannello: OLED SSD1309/SH1106 0x3C, e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 -> 10-wire ribbon to the front panel: OLED SSD1309/SH1106 0x3C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
- J7: Note Ventola 12 V 4 fili (cooler SP3/TR4) -> 12 V 4-wire fan (SP3/TR4 cooler)
- J8: Note 2x NTC 10k B3950 incollate allo spreader -> 2x NTC 10k B3950 glued to the spreader
- Q5: Note Invertitore ARM -> CLAMP -> ARM -> CLAMP inverter
- Q7: Note Open-drain PWM ventola (logica invertita in firmware) -> Open-drain fan PWM (inverted logic in firmware)
- R36: Note Tach su RX: scollegare la ventola se si programma via USB -> Tach on RX: unplug the fan when programming over USB
- R37: Note Bus esteso al pannello frontale (rev 0.3) -> Bus extended to the front panel (rev 0.3)
- R43: Note LED OUTPUT sul pannello: anodo a 3V3, catodo qui -> OUTPUT LED on the panel: anode to 3V3, cathode here
- R46: Note Pull-down: ARM basso = carico disabilitato -> Pull-down: ARM low = load disabled
- R47: Note Lettura ARM: 100k, un GPIO pilotato al boot non puo armare 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 -> ARM read-back: 100k, a GPIO driven at boot cannot arm the l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
- R53: Note NTC2 di riserva: il D1 mini ha un solo ADC (A0 = NTC1) -> NTC2 spare: the D1 mini has a single ADC (A0 = NTC1)
- U10: Note RSTSEL=0: reset a zero scala; LDAC=0: aggiornamento sincrono -> RSTSEL=0: reset to zero scale; LDAC=0: synchronous update
- U9: Note Espansore I2C @0x20; INT su GPIO0 (D3) -> I2C expander @0x20; INT on GPIO0 (D3)
Other:
- note added: "4-wire PWM fan and NTC sensors on the spreader"
- note added: "ARM / CLAMP logic (fail-safe: load off if the MCU is missing, in reset or faulty)"
- note added: "CLAMP high -> setpoints VSET1..4 shorted to ground"
- note added: "Front panel: I2C OLED, push encoder, OUTPUT button (rev 0.3)"
- note added: "Quad 16-bit DAC (internal 2.5 V reference)"
- note added: "WiFi module Wemos D1 mini Pro (ESP8266) on socket strips"
- note removed: "CLAMP alto -> setpoint VSET1..4 cortocircuitati a massa"
- note removed: "DAC quadruplo 16 bit (riferimento interno 2,5 V)"
- note removed: "Logica ARM / CLAMP (fail-safe: carico spento se MCU assente, in reset o in guasto)"
- note removed: "Modulo WiFi Wemos D1 mini Pro (ESP8266) su strip femmina"
- note removed: "Pannello frontale: OLED I2C, encoder con pulsante, tasto OUTPUT (rev 0.3)"
- note removed: "Ventola 4 fili PWM e sensori NTC sullo spreader"
- title: Carico attivo 60V 20A 300W — Controllo -> Electronic Load 4ch 60V 20A 300W — Control
