File: hardware/kicad/input.kicad_sch (KiCad schematic)
At the start: 24 parts, among them J1 DUT+, J2 DUT-, J3 SENSE, U1 TL431ID, U2 LM393

Commit message: Translate schematic and PCB to English
Sheets renamed (input, channels, control, power), all titles, notes,
values and board texts in English; symbol library renamed to eload.
Re-routed board: DRC with schematic parity clean.

Co-Authored-By: Claude Opus 5.5 <noreply@anthropic.com>
Claude-Session: https://claude.ai/code/session_013KrwoEq2Y4F9LNKutY5RJ4
Parts:
- D1: Note Inversione polarita: conduce e fa saltare F1 (verificare I2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 -> Reverse polarity: conducts and blows F1 (check I2t)
- F1: Note Fusibile lamellare ATO 25 A -> ATO blade fuse 25 A
- J1: Note Prigioniero M5, 25 A -> M5 stud, 25 A
- J2: Note Prigioniero M5, 25 A - punto stella di massa -> M5 stud, 25 A - ground star point
- R11: Note Soglia OTP ~100 C -> OTP threshold ~100 C
- R2: Note Fallback se il sense non e collegato -> Fallback when sense leads are not connected
- R3: Note SENSE- solo riferito a massa -> SENSE- referenced to ground only
- R6: Note Isteresi OVP -> OVP hysteresis
- R9: Note Isteresi OTP -> OTP hysteresis
Other:
- note added: "2.5 V reference and OVP / OTP comparators (open-collector outputs on ARM)"
- note added: "Comparator supply"
- note added: "DUT terminals and power-path protection"
- note added: "OTP: NTC 10k B3950 at ~100 C = 0.21 V < OTP_REF"
- note added: "OVP: trips at 2.5 V x (249k+10k)/10k = 64.7 V"
- note added: "Remote sense (voltage measured by the INA228s)"
- note removed: "Alimentazione comparatore"
- note removed: "Morsetti DUT e protezioni di potenza"
- note removed: "OTP: NTC 10k B3950 a ~100 C = 0,21 V < OTP_REF"
- note removed: "OVP: scatta a 2,5 V x (249k+10k)/10k = 64,7 V"
- note removed: "Remote sense (tensione misurata dagli INA228)"
- note removed: "Riferimento 2,5 V e comparatori OVP / OTP (uscite open-collector su ARM)"
- title: Carico attivo 60V 20A 300W — Ingresso e protezioni -> Electronic Load 4ch 60V 20A 300W — Input and protection
