File: hardware/kicad/power.kicad_sch (KiCad schematic)
At the start: 18 parts, among them J9 12V DC, U11 L78L05, U12 AP63205WU

Commit message: Translate schematic and PCB to English
Sheets renamed (input, channels, control, power), all titles, notes,
values and board texts in English; symbol library renamed to eload.
Re-routed board: DRC with schematic parity clean.

Co-Authored-By: Claude Opus 5.5 <noreply@anthropic.com>
Claude-Session: https://claude.ai/code/session_013KrwoEq2Y4F9LNKutY5RJ4
Parts:
- D5: value verde -> green
- F2: Note PTC 1206, hold 1,5 A (buck WiFi + ventola) -> PTC 1206, 1.5 A hold (WiFi buck + fan)
- U12: Note FB al 5 V di uscita (versione a uscita fissa) -> FB tied to the 5 V output (fixed-output version)
Other:
- note added: "+3V3 supplied by the Wemos module regulator (3V3 pin)"
- note added: "12 V auxiliary input (dedicated isolated adaptor) and regulators"
- note added: "Buck 12 V -> 5 V (AP63205) for the Wemos only: analog 5 V stays on the 78L05"
- note removed: "+3V3 fornita dal regolatore del modulo Wemos (pin 3V3)"
- note removed: "Buck 12 V -> 5 V (AP63205) solo per il Wemos: il 5 V analogico resta sul 78L05"
- note removed: "Ingresso ausiliario 12 V (alimentatore isolato dedicato) e regolatori"
- title: Carico attivo 60V 20A 300W — Alimentazione -> Electronic Load 4ch 60V 20A 300W — Power supplies
